File: STM32_CAN-USB.brd (EAGLE design)
At the start: 50 x 50 mm, 52 parts, among them IC1 STM32F105RBT, IC2 TJA1055T, IC3 BD9G101G, IC4 LM1117IMPX-3.3, Q1 16MHz, X1 MINI-USB

Commit message: change scheme, unrouted board
Parts:
- removed C15: 10uF, rcl:153CLV-0605
- removed C19, C22: 1nF, rcl:C0805
- removed C20, C23: 0.1, rcl:C0805
- removed C21, C24: 4.7uF, rcl:C0805
- removed D1: SS26, STM32_CAN-USB:SMB
- removed D2: SK36A, STM32_CAN-USB:DO-214AC
- removed DR2: CDRH3D16NP 6.8uH, STM32_CAN-USB:CDRH3D16NP
- removed F1: EST-157000 2A, STM32_CAN-USB:FUSE
- removed IC3: BD9G101G, STM32_CAN-USB:SSOP6
- added MC34063: MC34063, STM32_CAN-USB:SO8
- added R11: 3K, rcl:R0805
- C11: value 100uF/16v -> 10uF/16v; device rcl:153CLV-0605 -> rcl:SMC_A
- C12: value 0.015uF -> 220uF/35V; device rcl:C0805 -> rcl:153CLV-0810
- C13: value 0.1 -> 220pF
- C14: value 4.7uF/50v -> 220uF/35V; device rcl:153CLV-0605 -> rcl:153CLV-0810
- C16: value 10uF -> 220uF/16
- D3: value SM6T18CA -> SS14; device STM32_CAN-USB:DO214AA -> STM32_CAN-USB:SMA
- DR1: value CDRH127 100u -> 220uH
- R7: value 680 -> 0.33
- R8: value 3.9K -> 1K
- moved DR1 34.6 mm to (13.5, 35.0), turned to 0 degrees
- moved D3 25.1 mm to (21.5, 44.5), turned to 90 degrees
- moved R7 24.3 mm to (13.5, 49.5)
- moved C14 21.6 mm to (20.5, 54.5)
- moved C13 19.8 mm to (17.0, 47.0), turned to 90 degrees
- moved R8 17.8 mm to (9.00, 49.5)
- moved C12 15.3 mm to (10.5, 57.0), turned to 270 degrees
- moved IC4 6.10 mm to (36.5, 52.0)
- moved C16 5.10 mm to (29.0, 49.0)
- moved C11 3.64 mm to (38.0, 44.5), turned to 180 degrees
- moved C17 1.00 mm to (27.5, 42.5)
Connections:
- removed net N$17: C22.1, C23.1, C24.1, D2.A, D3.C, DR1.P$2
- net +12V: now also C12.+, MC34063.6, R7.1; no longer F1.P$1
- net +5V: now also C14.+, DR1.P$1, R11.1; no longer C13.2, C15.+, DR2.P$2, R8.1
- net BAT: no longer C14.+, D2.C, IC3.5
- net EN: no longer IC3.4
- net GND: now also C12.-, C13.2, MC34063.4, R8.2; no longer C15.-, C19.2, C20.2, C21.2, C22.2, C23.2, C24.2, D1.A, IC3.2, R7.1
- net N$12: now also MC34063.5, R11.2, R8.1; no longer C12.2, D1.C, DR2.P$1, IC3.6
- net N$13: now also D3.C, DR1.P$2, MC34063.2; no longer C13.1, IC3.3, R7.2, R8.2
- net N$18: now also C13.1, MC34063.3; no longer C19.1, C20.1, C21.1, DR1.P$1, F1.P$2
- net N$9: now also MC34063.1, MC34063.7, MC34063.8, R7.2; no longer C12.1, IC3.1
Routing:
- net BAT: track 53.5 -> 0.00 mm, vias 3 -> 0
- net +12V: track 23.8 -> 0.00 mm
- net N$17: track 22.3 -> 0.00 mm
- net EN: track 20.6 -> 0.35 mm, vias 2 -> 0
- net N$18: track 21.5 -> 3.07 mm
- net GND: track 120.1 -> 102.3 mm, vias 11 -> 1
- net +5V: track 70.5 -> 52.9 mm, vias 6 -> 4
- net +3V3: track 125.0 -> 138.9 mm
- net N$13: track 12.2 -> 22.6 mm
- net N$9: track 3.50 -> 1.27 mm
- removed copper zone on layer 1, net +5V
- removed copper zone on layer 1, net BAT
- removed copper zone on layer 1, net N$12
Other:
- board size 50 x 50 mm -> 50 x 59.5 mm

Commit message: TJA networks names
Connections:
- net N$14 renamed TJA_EN
- net N$15 renamed TJA_ERR
- net N$4 renamed TJA_RXD
- net N$5 renamed TJA_TXD
- net N$6 renamed TJA_STB
Changed lines of the file:
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@@
 <wire x1="42.35" y1="54.65" x2="39.5" y2="44.5" width="0.8128" layer="1"/>
 </signal>
-<signal name="N$4">
+<signal name="TJA_RXD">
 <contactref element="IC2" pad="3"/>
 <contactref element="IC1" pad="61"/>
@@
 <contactref element="R4" pad="2"/>
 </signal>
-<signal name="N$14">
+<signal name="TJA_EN">
 <contactref element="IC2" pad="6"/>
 <wire x1="32.4" y1="29.4" x2="32.4" y2="28.15" width="0.254" layer="1"/>
@@
 <wire x1="30.75" y1="26.5" x2="32.4" y2="28.15" width="0.254" layer="1"/>
 </signal>
-<signal name="N$6">
+<signal name="TJA_STB">
 <contactref element="IC2" pad="5"/>
 <wire x1="31.13" y1="29.4" x2="31.13" y2="27.88" width="0.254" layer="1"/>
@@
 <wire x1="30.25" y1="27" x2="31.13" y2="27.88" width="0.254" layer="1"/>
 </signal>
-<signal name="N$15">
+<signal name="TJA_ERR">
 <contactref element="IC2" pad="4"/>
 <contactref element="IC1" pad="57"/>
@@
 <wire x1="29.86" y1="28.36" x2="29.75" y2="28.25" width="0.254" layer="1"/>
 </signal>
-<signal name="N$5">
+<signal name="TJA_TXD">
 <contactref element="IC1" pad="62"/>
 <contactref element="IC2" pad="2"/>
