File: STM32_CAN-USB.sch (EAGLE design)
At the start: 52 parts, among them IC1 STM32F105RBT, IC2 TJA1055T, IC3 BD9G101G, IC4 LM1117IMPX-3.3, Q1 16MHz, X1 MINI-USB

Commit message: change scheme, unrouted board
Parts:
- removed C15: 10uF, rcl:CPOL-US153CLV-0605
- removed C19, C22: 1nF, rcl:C-EUC0805
- removed C20, C23: 0.1, rcl:C-EUC0805
- removed C21, C24: 4.7uF, rcl:C-EUC0805
- removed D1: SS26, STM32_CAN-USB:SCHOTTKY-DIODESMD
- removed D2: SK36A, STM32_CAN-USB:SK36A
- removed DR2: CDRH3D16NP 6.8uH, STM32_CAN-USB:CDRH3D16NP
- removed F1: EST-157000 2A, STM32_CAN-USB:FUSE
- removed IC3: BD9G101G, STM32_CAN-USB:BD9G101G
- added MC34063: MC34063, STM32_CAN-USB:MC34063
- added R11: 3K, rcl:R-EU_R0805
- C11: value 100uF/16v -> 10uF/16v; device rcl:CPOL-US153CLV-0605 -> rcl:CPOL-EUSMCA
- C12: value 0.015uF -> 220uF/35V; device rcl:C-EUC0805 -> rcl:CPOL-EU153CLV-0810
- C13: value 0.1 -> 220pF
- C14: value 4.7uF/50v -> 220uF/35V; device rcl:CPOL-US153CLV-0605 -> rcl:CPOL-EU153CLV-0810
- C16: value 10uF -> 220uF/16
- D3: value SM6T18CA -> SS14; device STM32_CAN-USB:SM6T18CA -> STM32_CAN-USB:SS14
- DR1: value CDRH127 100u -> 220uH
- R7: value 680 -> 0.33
- R8: value 3.9K -> 1K
Connections:
- removed net N$17: C22.1, C23.1, C24.1, D2.A, D3.2, DR1.2
- net +12V: now also C12.+, MC34063.VIN, R7.1; no longer F1.1
- net +5V: now also C14.+, DR1.1, R11.1; no longer C13.2, C15.+, DR2.2, R8.1
- net BAT: no longer C14.+, D2.C, IC3.VCC
- net EN: no longer IC3.EN
- net GND: now also C12.-, C13.2, D3.A, MC34063.GND, R8.2; no longer C15.-, C19.2, C20.2, C21.2, C22.2, C23.2, C24.2, D1.A, D3.1, IC3.GND, R7.1
- net N$12: now also MC34063.CMPR, R11.2, R8.1; no longer C12.2, D1.C, DR2.1, IC3.LX
- net N$13: now also D3.C, DR1.2, MC34063.SWE; no longer C13.1, IC3.FB, R7.2, R8.2
- net N$18: now also C13.1, MC34063.CT; no longer C19.1, C20.1, C21.1, DR1.1, F1.2
- net N$9: now also MC34063.DRVC, MC34063.IPK, MC34063.SWC, R7.2; no longer C12.1, IC3.BST
Other:
- moved on the sheet: C11, C13, C14, C16, C17, C18, DR1, IC4, JP1, R7, R8

Commit message: TJA networks names
Connections:
- net N$14 renamed TJA_EN
- net N$15 renamed TJA_ERR
- net N$4 renamed TJA_RXD
- net N$5 renamed TJA_TXD
- net N$6 renamed TJA_STB
Changed lines of the file:
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@@
 <?xml version="1.0" encoding="utf-8"?>
 <!DOCTYPE eagle SYSTEM "eagle.dtd">
-<eagle version="7.2.0">
+<eagle version="7.1.0">
 <drawing>
 <settings>
@@
 </segment>
 </net>
-<net name="N$4" class="0">
+<net name="TJA_RXD" class="0">
 <segment>
 <pinref part="IC2" gate="G$1" pin="RXD"/>
@@
 </segment>
 </net>
-<net name="N$14" class="0">
+<net name="TJA_EN" class="0">
 <segment>
 <pinref part="IC2" gate="G$1" pin="EN"/>
@@
 </segment>
 </net>
-<net name="N$6" class="0">
+<net name="TJA_STB" class="0">
 <segment>
 <pinref part="IC2" gate="G$1" pin="STB"/>
@@
 </segment>
 </net>
-<net name="N$15" class="0">
+<net name="TJA_ERR" class="0">
 <segment>
 <pinref part="IC2" gate="G$1" pin="ERR"/>
@@
 </segment>
 </net>
-<net name="N$5" class="0">
+<net name="TJA_TXD" class="0">
 <segment>
 <pinref part="IC2" gate="G$1" pin="TXD"/>
