File: Eagle/STM32_CAN-USB.brd (EAGLE design)
At the start: 50 x 59.5 mm, 42 parts, among them IC1 STM32F105RBT, IC2 TJA1055T, IC4 LM1117IMPX-3.3, Q1 16MHz, X1 MINI-USB

Commit message: Revert sch & brd
Parts:
- removed MC34063: MC34063, STM32_CAN-USB:SO8
- removed R11: 3K, rcl:R0805
- added C15: 10uF, rcl:153CLV-0605
- added C19, C22: 1nF, rcl:C0805
- added C20, C23: 0.1, rcl:C0805
- added C21, C24: 4.7uF, rcl:C0805
- added D1: SS26, STM32_CAN-USB:SMB
- added D2: SK36A, STM32_CAN-USB:DO-214AC
- added DR2: CDRH3D16NP 6.8uH, STM32_CAN-USB:CDRH3D16NP
- added F1: EST-157000 2A, STM32_CAN-USB:FUSE
- added IC3: BD9G101G, STM32_CAN-USB:SSOP6
- C11: value 10uF/16v -> 100uF/16v; device rcl:SMC_A -> rcl:153CLV-0605
- C12: value 220uF/35V -> 0.015uF; device rcl:153CLV-0810 -> rcl:C0805
- C13: value 220pF -> 0.1
- C14: value 220uF/35V -> 4.7uF/50v; device rcl:153CLV-0810 -> rcl:153CLV-0605
- C16: value 220uF/16 -> 10uF
- D3: value SS14 -> SM6T18CA; device STM32_CAN-USB:SMA -> STM32_CAN-USB:DO214AA
- DR1: value 220uH -> CDRH127 100u
- R7: value 0.33 -> 680
- R8: value 1K -> 3.9K
- moved DR1 34.6 mm to (48.0, 33.0), turned to 180 degrees
- moved D3 25.1 mm to (46.5, 47.0), turned to 180 degrees
- moved R7 24.3 mm to (10.0, 25.5)
- moved C14 21.6 mm to (16.5, 33.2)
- moved C13 19.8 mm to (10.0, 28.5), turned to 0 degrees
- moved R8 17.8 mm to (10.0, 31.8)
- moved C12 15.3 mm to (10.0, 41.8), turned to 0 degrees
- moved IC4 6.10 mm to (31.5, 48.5)
- moved C16 5.10 mm to (24.0, 48.0)
- moved C11 3.64 mm to (39.0, 48.0), turned to 90 degrees
- moved C17 1.00 mm to (26.5, 42.5)
Connections:
- net TJA_EN renamed N$14
- net TJA_ERR renamed N$15
- net TJA_RXD renamed N$4
- net TJA_STB renamed N$6
- net TJA_TXD renamed N$5
- new net N$17: C22.1, C23.1, C24.1, D2.A, D3.C, DR1.P$2
- net +12V: now also F1.P$1; no longer C12.+, MC34063.6, R7.1
- net +5V: now also C13.2, C15.+, DR2.P$2, R8.1; no longer C14.+, DR1.P$1, R11.1
- net BAT: now also C14.+, D2.C, IC3.5
- net EN: now also IC3.4
- net GND: now also C15.-, C19.2, C20.2, C21.2, C22.2, C23.2, C24.2, D1.A, IC3.2, R7.1; no longer C12.-, C13.2, MC34063.4, R8.2
- net N$12: now also C12.2, D1.C, DR2.P$1, IC3.6; no longer MC34063.5, R11.2, R8.1
- net N$13: now also C13.1, IC3.3, R7.2, R8.2; no longer D3.C, DR1.P$2, MC34063.2
- net N$18: now also C19.1, C20.1, C21.1, DR1.P$1, F1.P$2; no longer C13.1, MC34063.3
- net N$9: now also C12.1, IC3.1; no longer MC34063.1, MC34063.7, MC34063.8, R7.2
Routing:
- net BAT: track 0.00 -> 53.5 mm, vias 0 -> 3
- net +12V: track 0.00 -> 23.8 mm
- net N$17: track 0.00 -> 22.3 mm
- net EN: track 0.35 -> 20.6 mm, vias 0 -> 2
- net N$18: track 3.07 -> 21.5 mm
- net GND: track 102.3 -> 120.1 mm, vias 1 -> 11
- net +5V: track 52.9 -> 70.5 mm, vias 4 -> 6
- net +3V3: track 138.9 -> 125.0 mm
- net N$13: track 22.6 -> 12.2 mm
- net N$9: track 1.27 -> 3.50 mm
- added copper zone on layer 1, net +5V
- added copper zone on layer 1, net BAT
- added copper zone on layer 1, net N$12
Other:
- board size 50 x 59.5 mm -> 50 x 50 mm
